File: PCB/Can and power/Can and power.kicad_pcb (KiCad board)
At the start: 4 copper layers, 43.4 x 43.5 mm, 39 parts, among them J1 TPS54232DR, J3 HDR_143_1, J4 HDR_143_2, J5 SKT_146, J6 HDR_175, J7 Car connector, U1 SN65HVD230

Commit message: Position refinements
Parts:
- J5: footprint Connector_PinSocket_1.27mm:PinSocket_2x10_P1.27mm_Vertical -> Project_footprints:PinSocket_2x10_P1.27mm_Vertical_CA
- moved J5 5.75 mm to (151.2, 91.1)

Commit message: v6.1 placeholder for bulk resistor and capacitor
Parts:
- added C12: 0.1uF 50V, Capacitor_SMD:C_1206_3216Metric, F.Cu at (136.7, 97.0)
- added R11: 100, Resistor_SMD:R_1206_3216Metric, F.Cu at (132.9, 94.7)
- J5: footprint Project_footprints:PinSocket_2x10_P1.27mm_Vertical_CA -> Connector_PinSocket_1.27mm:PinSocket_2x10_P1.27mm_Vertical
- moved J5 5.75 mm to (147.1, 87.0)
- moved F1 1.17 mm to (136.7, 94.0), turned to 180 degrees
Routing:
- added copper zone on F.Cu, net Net-(C12-Pad1)

Commit message: LCSC BOM finalisation
Parts:
- D4: value 2V-20mA -> 2V - 20mA
- R11: value 100 -> 100R

Commit message: Production order v6.1
Routing:
- net +3V3: track 76.7 -> 77.3 mm
