File: PCB/Can and power/Can and power.kicad_pcb (KiCad board)
At the start: 4 copper layers, 43.4 x 43.5 mm, 41 parts, among them J1 TPS54232DR, J3 HDR_143_1, J4 HDR_143_2, J5 SKT_146, J6 HDR_175, J7 Car connector, U1 SN65HVD230

Commit message: CAN connector changed to PH
Parts:
- J7: footprint Connector_JST:JST_EH_B4B-EH-A_1x04_P2.50mm_Vertical -> Connector_JST:JST_PH_B4B-PH-K_1x04_P2.00mm_Vertical
- moved D2 0.43 mm to (133.5, 103.4)
- moved D1 0.35 mm to (133.4, 101.2)
- moved J7 0.29 mm to (137.5, 101.5)
- moved C6 0.25 mm to (140.8, 99.5)
Routing:
- net /CAN_L: track 11.7 -> 10.6 mm
- net GND: vias 198 -> 195
