File: PCB/Can and power/Can and power.kicad_sch (KiCad schematic)
At the start: 41 parts, among them J1 TPS54232DR, J3 HDR_143_1, J4 HDR_143_2, J5 SKT_146, J6 HDR_175, J7 Car connector, U1 SN65HVD230

Commit message: CAN connector changed to PH
Parts:
- J7: footprint Connector_JST:JST_EH_B4B-EH-A_1x04_P2.50mm_Vertical -> Connector_JST:JST_PH_B4B-PH-K_1x04_P2.00mm_Vertical; LCSC C160258 -> C265289; LCSC alt. C160258 -> C265289; Manufacturer_Part_Number B4B-EH-A -> B4B-PH-K(LF)(SN)
Changed lines of the file:
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@@
 			)
 		)
-		(property "Footprint" "Connector_JST:JST_EH_B4B-EH-A_1x04_P2.50mm_Vertical"
+		(property "Footprint" "Connector_JST:JST_PH_B4B-PH-K_1x04_P2.00mm_Vertical"
 			(at 267.97 43.18 0)
 			(effects
@@
 			)
 		)
-		(property "Datasheet" "https://www.jst-mfg.com/product/pdf/eng/eEH.pdf"
+		(property "Datasheet" "https://www.lcsc.com/datasheet/C265289.pdf?spm=wm.fly.bg.1.pdf___wm.ssy.ml.0-0-0.ent&lcsc_vid=RAdcUQIHEwRdBlMATwJdUVJeFlVXBF1eTwUNBVJUFFgxVlNeQlBZU11TT1RdUjsOAxUeFF5JWBYZEEoKFBINSQcJGk4%3D"
 			(at 267.97 43.18 0)
 			(effects
@@
 			)
 		)
-		(property "Manufacturer_Part_Number" "B4B-EH-A"
+		(property "Manufacturer_Part_Number" "B4B-PH-K(LF)(SN)"
 			(at 267.97 52.07 0)
 			(effects
@@
 			)
 		)
-		(property "LCSC alt." "C160258"
+		(property "LCSC alt." "C265289"
 			(at 267.97 43.18 0)
 			(effects
@@
 			)
 		)
-		(property "LCSC" "C160258"
+		(property "LCSC" "C265289"
 			(at 267.97 43.18 0)
 			(effects
